Commit message: section 4

File: bumperbot_ws/src/bumperbot_description/urdf/bumperbot.urdf.xacro (robot description, xacro)
@@ -1,6 +1,14 @@
 <?xml version="1.0"?>
-<robot name="bumperbot">
+<robot name="bumperbot" xmlns:xacro="http://ros.org/wiki/xacro">
+  <xacro:include filename="$(find bumperbot_description)/urdf/bumperbot_gazebo.xacro"/>
   <link name="base_footprint"/>
   <link name="base_link">
+    <inertial>
+      <origin xyz="0 0 0.04" rpy="0.0 0.25 0.3" />
+      <mass value="8.2573504e-01"/>
+      <inertia ixx="2.2124416e-02" ixy="-1.2294101e-04" ixz="3.4938785e-04"
+               iyy="2.1193702e-02" iyz="-5.0120904e-05"
+               izz="2.0064271e-02" />
+    </inertial>
     <visual>
         <origin rpy="0 0 0" xyz="0 0 0"/>
@@ -22,4 +30,11 @@
   </joint>
   <link name="wheel_right_link">
+    <inertial>
+      <origin xyz="0 -0.014 0" rpy="0 0 0" />
+      <mass value="0.0530086090966721" />
+      <inertia ixx="1.88176298336665E-05" ixy="-4.8444933029987E-10" ixz="1.88163708851143E-08"
+               iyy="3.11510738647764E-05" iyz="-6.93560663069607E-11"
+               izz="1.8801969558182E-05" />
+    </inertial>
     <visual>
         <origin rpy="1.57 0 0" xyz="0 0 0"/>
@@ -28,4 +43,10 @@
         </geometry>
     </visual>
+    <collison>
+      <origin xyz="0 -0.015 0" rpy="1.57.0.0"/>
+      <geometry>
+        <sphere radius="0.033"/>
+      </geometry>
+    </collison>
   </link>
   <joint name="wheel_right_joint" type="continuous">
@@ -36,4 +57,11 @@
   </joint>
   <link name="wheel_left_link">
+    <inertial>
+      <origin xyz="0 0.014 0" rpy="0 0 0" />
+      <mass value="0.0530086043217644" />
+      <inertia ixx="1.8792911368909E-05"  ixy="3.31256392204584E-10" ixz="-1.14082001662767E-08"
+               iyy="3.11510738759073E-05" iyz="-3.60499245082192E-10"
+               izz="1.88266886146847E-05" />
+    </inertial>
     <visual>
         <origin rpy="-1.57 0 0" xyz="0 0 0"/>
@@ -42,4 +70,10 @@
         </geometry>
     </visual>
+    <collison>
+      <origin xyz="0 0.015 0" rpy="1.57 0 0"/>
+      <geometry>
+        <sphere radius="0.033"/>
+      </geometry>
+    </collison>
   </link>
   <joint name="wheel_left_joint" type="continuous">
@@ -50,4 +84,11 @@
   </joint>
   <link name="caster_front_link">
+    <inertial>
+      <origin xyz="3.89968128948481E-07 2.40073004698083E-07 0.00219173397061506" rpy="0 0 0" />
+      <mass value="1.44379265037903E-06" />
+      <inertia ixx="7.23075276010246E-11" ixy="-6.10956883467859E-16" ixz="2.22849693525031E-15"
+               iyy="3.8713793085917E-11"  iyz="2.93909858781952E-15"
+               izz="1.00967486676306E-10" />
+    </inertial>
     <visual>
         <origin rpy="0 0 0" xyz="0 0 0"/>
@@ -56,4 +97,10 @@
         </geometry>
     </visual>
+    <collison>
+      <origin xyz="0 0 0" rpy="0 0 0"/>
+      <geometry>
+        <sphere radius="0.005"/>
+      </geometry>
+    </collison>
   </link>
   <joint name="caster_front_joint" type="fixed">
@@ -63,4 +110,11 @@
   </joint>
   <link name="caster_rear_link">
+    <inertial>
+      <origin xyz="3.8996812895542E-07 2.40073004698083E-07 0.00219173397061509" rpy="0 0 0" />
+      <mass value="1.44379265037902E-06" />
+      <inertia ixx="7.23075276010246E-11" ixy="-6.10956872363424E-16" ixz="2.22849693527207E-15"
+               iyy="3.87137930859167E-11" iyz="2.939098587861E-15"
+               izz="1.00967486676306E-10" />
+    </inertial>
     <visual>
         <origin rpy="0 0 0" xyz="0 0 0"/>
@@ -69,4 +123,10 @@
         </geometry>
     </visual>
+    <collison>
+      <origin xyz="0 0 0" rpy="0 0 0"/>
+      <geometry>
+        <sphere radius="0.005"/>
+      </geometry>
+    </collison>
   </link>
   <joint name="caster_rear_joint" type="fixed">

Commit message: secao 5

File: bumperbot_ws/src/bumperbot_description/urdf/bumperbot.urdf.xacro (robot description, xacro)
@@ -12,13 +12,13 @@
     </inertial>
     <visual>
-        <origin rpy="0 0 0" xyz="0 0 0"/>
-        <geometry>
-            <mesh filename="package://bumperbot_description/meshes/base_link.STL"/>
-        </geometry>
+      <origin xyz="0 0 0" rpy="0 0 0" />
+      <geometry>
+        <mesh filename="package://bumperbot_description/meshes/base_link.STL" />
+      </geometry>
     </visual>
     <collision>
-      <origin rpy="0 0 0" xyz="0 0 0"/>
+      <origin xyz="0 0 0" rpy="0 0 0" />
       <geometry>
-          <mesh filename="package://bumperbot_description/meshes/base_link.STL"/>
+        <mesh filename="package://bumperbot_description/meshes/base_link.STL" />
       </geometry>
     </collision>
@@ -26,6 +26,6 @@
   <joint name="base_joint" type="fixed">
     <parent link="base_footprint"/>
-    <child link="base_link"/>
-    <origin rpy="0 0 0" xyz="0 0 0.033"/>
+    <child link="base_link" />
+    <origin xyz="0 0 0.033" rpy="0 0 0"/>
   </joint>
   <link name="wheel_right_link">
@@ -38,23 +38,24 @@
     </inertial>
     <visual>
-        <origin rpy="1.57 0 0" xyz="0 0 0"/>
-        <geometry>
-            <mesh filename="package://bumperbot_description/meshes/wheel_right_link.STL"/>
-        </geometry>
+      <origin xyz="0 0 0" rpy="1.57 0 0" />
+      <geometry>
+        <mesh filename="package://bumperbot_description/meshes/wheel_right_link.STL" />
+      </geometry>
     </visual>
-    <collison>
-      <origin xyz="0 -0.015 0" rpy="1.57.0.0"/>
+    <collision>
+      <origin xyz="0 -0.015 0" rpy="1.57 0 0" />
       <geometry>
         <sphere radius="0.033"/>
       </geometry>
-    </collison>
+    </collision>
   </link>
   <joint name="wheel_right_joint" type="continuous">
-    <origin rpy="0 0 0" xyz="0 -0.07 0"/>
-    <parent link="base_link"/>
-    <child link="wheel_right_link"/>
-    <axis xyz="0 1 0"/>
+    <origin xyz="0 -0.0701101849418637 0" rpy="0 0 0" />
+    <parent link="base_link" />
+    <child link="wheel_right_link" />
+    <axis xyz="0 1 0" />
   </joint>
-  <link name="wheel_left_link">
+  <link
+    name="wheel_left_link">
     <inertial>
       <origin xyz="0 0.014 0" rpy="0 0 0" />
@@ -65,21 +66,21 @@
     </inertial>
     <visual>
-        <origin rpy="-1.57 0 0" xyz="0 0 0"/>
-        <geometry>
-            <mesh filename="package://bumperbot_description/meshes/wheel_left_link.STL"/>
-        </geometry>
+      <origin xyz="0 0 0" rpy="-1.57 0 0" />
+      <geometry>
+        <mesh filename="package://bumperbot_description/meshes/wheel_left_link.STL" />
+      </geometry>
     </visual>
-    <collison>
-      <origin xyz="0 0.015 0" rpy="1.57 0 0"/>
+    <collision>
+      <origin xyz="0 0.015 0" rpy="-1.57 0 0" />
       <geometry>
         <sphere radius="0.033"/>
       </geometry>
-    </collison>
+    </collision>
   </link>
   <joint name="wheel_left_joint" type="continuous">
-    <origin rpy="0 0 0" xyz="0 0.07 0"/>
-    <parent link="base_link"/>
-    <child link="wheel_left_link"/>
-    <axis xyz="0 1 0"/>
+    <origin xyz="0 0.0701101849418642 0" rpy="0 0 0" />
+    <parent link="base_link" />
+    <child link="wheel_left_link" />
+    <axis xyz="0 1 0" />
   </joint>
   <link name="caster_front_link">
@@ -92,20 +93,21 @@
     </inertial>
     <visual>
-        <origin rpy="0 0 0" xyz="0 0 0"/>
-        <geometry>
-            <mesh filename="package://bumperbot_description/meshes/caster_front_link.STL"/>
-        </geometry>
+      <origin xyz="0 0 0" rpy="0 0 0" />
+      <geometry>
+        <mesh filename="package://bumperbot_description/meshes/caster_front_link.STL" />
+      </geometry>
     </visual>
-    <collison>
-      <origin xyz="0 0 0" rpy="0 0 0"/>
+    <collision>
+      <origin xyz="0 0 0" rpy="0 0 0" />
       <geometry>
         <sphere radius="0.005"/>
       </geometry>
-    </collison>
+    </collision>
   </link>
   <joint name="caster_front_joint" type="fixed">
-    <origin rpy="0 0 0" xyz="0.0475 0 -0.0275"/>
-    <parent link="base_link"/>
-    <child link="caster_front_link"/>
+    <origin xyz="0.04755 0 -0.0275" rpy="0 0 0" />
+    <parent link="base_link" />
+    <child link="caster_front_link" />
+    <axis xyz="0 0 0" />
   </joint>
   <link name="caster_rear_link">
@@ -118,33 +120,21 @@
     </inertial>
     <visual>
-        <origin rpy="0 0 0" xyz="0 0 0"/>
-        <geometry>
-            <mesh filename="package://bumperbot_description/meshes/caster_rear_link.STL"/>
-        </geometry>
+      <origin xyz="0 0 0" rpy="0 0 0" />
+      <geometry>
+        <mesh filename="package://bumperbot_description/meshes/caster_rear_link.STL" />
+      </geometry>
     </visual>
-    <collison>
-      <origin xyz="0 0 0" rpy="0 0 0"/>
+    <collision>
+      <origin xyz="0 0 0" rpy="0 0 0" />
       <geometry>
         <sphere radius="0.005"/>
       </geometry>
-    </collison>
+    </collision>
   </link>
   <joint name="caster_rear_joint" type="fixed">
-    <origin rpy="0 0 0" xyz="-0.0475 0 -0.0275"/>
-    <parent link="base_link"/>
-    <child link="caster_rear_link"/>
-  </joint>
-  <link name="camera_link">
-    <visual>
-        <origin xyz="-0.03 0.03 0" rpy="1.57 0 0"/>
-        <geometry>
-            <mesh filename="package://bumperbot_description/meshes/camera_link.STL"/>
-        </geometry>
-    </visual>
-  </link>
-  <joint name="camera_joint" type="fixed">
-    <origin rpy="0 0 0" xyz="0 0 0"/>
-    <parent link="base_link"/>
-    <child link="camera_link"/>
+    <origin xyz="-0.04755 0 -0.0275" rpy="0 0 0" />
+    <parent link="base_link" />
+    <child link="caster_rear_link" />
+    <axis xyz="0 0 0" />
   </joint>
 </robot>

File: bumperbot_ws/src/bumperbot_description/urdf/bumperbot_gazebo.xacro (robot description, xacro)
@@ -1,4 +1,24 @@
 <?xml version="1.0"?>
-<robot name="bumperbot" xmlns="http://ros.org/wiki/xacro">
+<robot name="bumperbot" xmlns:xacro="http://ros.org/wiki/xacro">
+  <transmission name="wheel_right_transmission">
+    <type>transmission_interface/SimpleTransmission</type>
+    <joint name="wheel_right_joint" >
+      <hardwareInterface>hardware_interface/VelocityJointInterface</hardwareInterface>
+    </joint>
+    <actuator name="wheel_right_motor" >
+      <hardwareInterface>hardware_interface/VelocityJointInterface</hardwareInterface>
+      <mechanicalReduction>1.0</mechanicalReduction>
+    </actuator>
+  </transmission>
+  <transmission name="wheel_left_transmission">
+    <type>transmission_interface/SimpleTransmission</type>
+    <joint name="wheel_left_joint" >
+      <hardwareInterface>hardware_interface/VelocityJointInterface</hardwareInterface>
+    </joint>
+    <actuator name="wheel_left_motor" >
+      <hardwareInterface>hardware_interface/VelocityJointInterface</hardwareInterface>
+      <mechanicalReduction>1.0</mechanicalReduction>
+    </actuator>
+  </transmission>
   <gazebo reference="wheel_left_link">
     <mu1>1000000000000000.0</mu1>
@@ -35,3 +55,10 @@
     <maxVel>1.0</maxVel>
   </gazebo>
+  <!-- ROS Control -->
+  <gazebo>
+    <plugin name="gazebo_ros_control" filename="libgazebo_ros_control.so">
+      <robotSimType>gazebo_ros_control/DefaultRobotHWSim</robotSimType>
+      <legacyModeNS>true</legacyModeNS>
+    </plugin>
+  </gazebo>
 </robot>
